File: Hardware/10MHz-amp/10MHz-amp.kicad_sch (KiCad schematic)
At the start: 138 parts, among them J1 Conn_Coaxial, J10 1x03_Socket, J11 1x03_Socket, J12 01x03_Pin, J13 Conn_01x08_Socket, J14 Conn_01x08_Pin, J2 BANANA_JACK, J3 BANANA_JACK, J4 BANANA_JACK, J5 1x03_Socket, J6 Conn_01x03_Pin, J7 Conn_Coaxial, J8 PJ-063AH, J9 Conn_01x03_Pin, K1 TQ2-24V, K2 TQ2-24V, K3 TQ2-24V, K4 TQ2-24V, K5 TQ2-24V, K6 TQ2-24V, Q1 DMPH6250SQ-13, Q2 DMN6075SQ-7, Q3 DMPH6250SQ-13, SW1 SW_SPDT, SW2 SW_SPDT, SW3 SW_SPDT, SW4 SP6T-A10603RNZQ, U1 THS3491xDDA

Commit message: added values for 50Ohm term resistors and updated gain resistor values
Parts:
- removed R14: 50R, Resistor_SMD:R_0603_1608Metric, symbol Device:R
- removed R7: 1R, Resistor_SMD:R_0603_1608Metric, symbol Device:R
- added C24, C27: 1000p, Capacitor_SMD:C_0603_1608Metric, symbol Device:C
- added C25, C26: 100p, Capacitor_SMD:C_0603_1608Metric, symbol Device:C
- added HS2: Heatsink, symbol Mechanical:Heatsink
- added RxL, RxS: 50R, symbol Device:R
- added RxO: 1M, symbol Device:R
- added T1: TLINE, symbol Simulation_SPICE:TLINE
- added V1: VSIN, symbol Simulation_SPICE:VSIN
- R1: Manufactor Part Number PTN16-A01120K1C1 -> PTN16-A01115K1A1; Notes REVERSE LOG -> LOG; Supplier Link https://www.digikey.co.nz/en/products/detail/same-sky-formerly-cui-devices/PTN16-A01120K1C1/20380778 -> https://www.digikey.co.nz/en/products/detail/same-sky-formerly-cui-devices/PTN16-A01115K1A1/20380947; Supplier Part Number 2223-PTN16-A01120K1C1-ND -> 2223-PTN16-A01115K1A1-ND; Supplier link https://www.digikey.co.nz/en/products/detail/same-sky-formerly-cui-devices/PTN16-A01120K1C1/20380778 -> https://www.digikey.co.nz/en/products/detail/same-sky-formerly-cui-devices/PTN16-A01115K1A1/20380947
- R12: value 1000R -> 3000R
- R2: value 1k -> 1000R
- R3: value 200R -> 274R
- R4: value 110R -> 157R
- R5: value 10R2 -> 15R0
- R6: value 1R -> 50R; Manufactor Part Number (none) -> PWR163S-25-50R0FE; Notes (none) -> 18w; Supplier Part Number (none) -> 118-PWR163S-25-50R0FECT-ND; Supplier link (none) -> https://www.digikey.co.nz/en/products/detail/bourns-inc/PWR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
- R8: Manufactor Part Number (none) -> PWR163S-25-50R0FE; Supplier Part Number (none) -> 118-PWR163S-25-50R0FECT-ND; Supplier link (none) -> https://www.digikey.co.nz/en/products/detail/bourns-inc/PWR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
Connections:
- net FO_HS: now also R6.2
- net GND: now also C24.2, C25.2, C26.2, C27.2, RxL.1, RxO.1, T1.2, T1.4, V1.2
- net O_HS: now also R6.1
- net VCC: now also C26.1, C27.1
- net VS: now also C24.1, C25.1
- net at R4.1: now also K4.3; no longer R6.2
- net at K1.3: now also R1.1
- new net: RxL.2, RxO.2, T1.3
- new net: RxS.1, V1.1
- new net: RxS.2, T1.1
Other:
- note added: "50"
- note added: "50 + 50"
- note added: "= Vso"
- note added: "= Vso * 1/2"
- note added: "AMP IN = Vsi"
- note added: "BECAUSE WE WANT THE OUTPUT VOLTAGE OF THE AMP TO BE SOME GAIN OF THE OUTPUT OF THE FUNCTION GEN AND THE INCOMING VOLTAGE IS HALFED DUE TO THE VOLTAGE DIVIDER FORMED BY RxS and RxL. THAT MEANS ALL GAINS NEED TO BE MULTIPLIED BY 2"
- note added: "BOTH RxS AND RxL CREATE A VOLTAGE DIVIDER THEREFORE:"
- note added: "FUNCTION GEN OUT = Vso"
- note added: "FUNCTIONAL DIAGRAM OF SYSTEM"
- note added: "RI = RF/(2A_G-1)"
- note added: "RxL"
- note added: "RxL+RxS"
- note added: "Vsi"
- note added: "Vsi = Vso"
- note added: "Vsi = Vso/2"
- note added: "Vso"
- note removed: "RI = RF/(A_G-1)"
- moved on the sheet: C4, C5, C6, R1, R2, R3, R4, R5

Commit message: updated function diagram of system input
Parts:
- added FB4, FB5: 2508051217Y6, Resistor_SMD:R_0805_2012Metric, symbol Device:FerriteBead
- C1: renamed from C26; Manufactor Part Number C0603C103K5RACTU -> CC0603KPX7R9BB101; Supplier Part Number 399-C0603C103K5RACTUCT-ND -> 13-CC0603KPX7R9BB101CT-ND; Supplier link https://www.digikey.co.nz/en/products/detail/kemet/C0603C10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 -> https://www.digikey.co.nz/en/products/detail/yageo/CC0603KP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
- C2: renamed from C27; Manufactor Part Number C0603C103K5RACTU -> C0603C102K5RACTU; Supplier Part Number 399-C0603C103K5RACTUCT-ND -> 399-C0603C102K5RACTUCT-ND; Supplier link https://www.digikey.co.nz/en/products/detail/kemet/C0603C103K5RACTU/411090 -> https://www.digikey.co.nz/en/products/detail/kemet/C0603C102K5RACTU/411081
- C6: renamed from C25; Manufactor Part Number C0603C103K5RACTU -> CC0603KPX7R9BB101; Supplier Part Number 399-C0603C103K5RACTUCT-ND -> 13-CC0603KPX7R9BB101CT-ND; Supplier link https://www.digikey.co.nz/en/products/detail/kemet/C0603C10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 -> https://www.digikey.co.nz/en/products/detail/yageo/CC0603KP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
- C7: renamed from C24; Manufactor Part Number C0603C103K5RACTU -> C0603C102K5RACTU; Supplier Part Number 399-C0603C103K5RACTUCT-ND -> 399-C0603C102K5RACTUCT-ND; Supplier link https://www.digikey.co.nz/en/products/detail/kemet/C0603C103K5RACTU/411090 -> https://www.digikey.co.nz/en/products/detail/kemet/C0603C102K5RACTU/411081
- R10: renamed from R12; footprint Resistor_SMD:R_0603_1608Metric -> Resistor_SMD:R_1206_3216Metric; Manufactor Part Number (none) -> RT0603DRD073KL; Notes (none) -> 25ppm; Supplier Part Number (none) -> 311-3.0KDCT-ND; Supplier link (none) -> https://www.digikey.co.nz/en/products/detail/yageo/RT0603DR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
- R11: renamed from R13; Manufactor Part Number (none) -> RT0603BRD0710KL; Supplier Part Number (none) -> YAG1236CT-ND; Supplier link (none) -> https://www.digikey.co.nz/en/products/detail/yageo/RT0603BR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
- R13: renamed from R15; Manufactor Part Number (none) -> RT0603BRD0710KL; Supplier Part Number (none) -> YAG1236CT-ND; Supplier link (none) -> https://www.digikey.co.nz/en/products/detail/yageo/RT0603BR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
- R14: renamed from R16; Manufactor Part Number (none) -> RT0603BRD0710KL; Supplier Part Number (none) -> YAG1236CT-ND; Supplier link (none) -> https://www.digikey.co.nz/en/products/detail/yageo/RT0603BR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
- R15: renamed from R17; Manufactor Part Number (none) -> RT0603BRD0710KL; Supplier Part Number (none) -> YAG1236CT-ND; Supplier link (none) -> https://www.digikey.co.nz/en/products/detail/yageo/RT0603BR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
- R16: renamed from R18; Manufactor Part Number (none) -> RC0603JR-070RL; Supplier Part Number (none) -> 311-0.0GRCT-ND; Supplier link (none) -> https://www.digikey.co.nz/en/products/detail/yageo/RC0603JR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
- R17: renamed from R19; Manufactor Part Number (none) -> RC0603JR-070RL; Supplier Part Number (none) -> 311-0.0GRCT-ND; Supplier link (none) -> https://www.digikey.co.nz/en/products/detail/yageo/RC0603JR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
- R18: renamed from R20; Manufactor Part Number (none) -> RC0603JR-070RL; Supplier Part Number (none) -> 311-0.0GRCT-ND; Supplier link (none) -> https://www.digikey.co.nz/en/products/detail/yageo/RC0603JR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
- R19: renamed from R21; Manufactor Part Number (none) -> RC0603JR-070RL; Supplier Part Number (none) -> 311-0.0GRCT-ND; Supplier link (none) -> https://www.digikey.co.nz/en/products/detail/yageo/RC0603JR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
- R2: Manufactor Part Number (none) -> RT0603BRC071KL; Notes (none) -> 15ppm; Supplier Part Number (none) -> YAG4454CT-ND; Supplier link (none) -> https://www.digikey.co.nz/en/products/detail/yageo/RT0603BR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
- R20: renamed from R22; Manufactor Part Number (none) -> RC0603JR-070RL; Supplier Part Number (none) -> 311-0.0GRCT-ND; Supplier link (none) -> https://www.digikey.co.nz/en/products/detail/yageo/RC0603JR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
- R21: renamed from R23; Manufactor Part Number (none) -> RT0603BRD0710KL; Supplier Part Number (none) -> YAG1236CT-ND; Supplier link (none) -> https://www.digikey.co.nz/en/products/detail/yageo/RT0603BR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
- R22: renamed from R24; Manufactor Part Number (none) -> RT0603BRD0710KL; Supplier Part Number (none) -> YAG1236CT-ND; Supplier link (none) -> https://www.digikey.co.nz/en/products/detail/yageo/RT0603BR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
- R23: renamed from R25; Manufactor Part Number (none) -> RT0603BRD0710KL; Supplier Part Number (none) -> YAG1236CT-ND; Supplier link (none) -> https://www.digikey.co.nz/en/products/detail/yageo/RT0603BR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
- R24: renamed from R26; Manufactor Part Number (none) -> RT0603BRD0710KL; Supplier Part Number (none) -> YAG1236CT-ND; Supplier link (none) -> https://www.digikey.co.nz/en/products/detail/yageo/RT0603BR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
- R25: renamed from R27; Manufactor Part Number (none) -> RT0603BRD0710KL; Supplier Part Number (none) -> YAG1236CT-ND; Supplier link (none) -> https://www.digikey.co.nz/en/products/detail/yageo/RT0603BR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
- R26: renamed from R28; Manufactor Part Number (none) -> RT0603BRD0710KL; Supplier Part Number (none) -> YAG1236CT-ND; Supplier link (none) -> https://www.digikey.co.nz/en/products/detail/yageo/RT0603BR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
- R27: renamed from R29; Manufactor Part Number (none) -> RT0603BRD0710KL; Supplier Part Number (none) -> YAG1236CT-ND; Supplier link (none) -> https://www.digikey.co.nz/en/products/detail/yageo/RT0603BR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
- R28: renamed from R30; Manufactor Part Number (none) -> RT0603BRD0710KL; Supplier Part Number (none) -> YAG1236CT-ND; Supplier link (none) -> https://www.digikey.co.nz/en/products/detail/yageo/RT0603BR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
- R29: renamed from R31; Manufactor Part Number (none) -> RC0603JR-070RL; Supplier Part Number (none) -> 311-0.0GRCT-ND; Supplier link (none) -> https://www.digikey.co.nz/en/products/detail/yageo/RC0603JR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
- R3: footprint Resistor_SMD:R_0603_1608Metric -> Resistor_SMD:R_0805_2012Metric; Manufactor Part Number (none) -> RT0805BRD07274RL; Notes (none) -> 25ppm; Supplier Part Number (none) -> YAG4868CT-ND; Supplier link (none) -> https://www.digikey.co.nz/en/products/detail/yageo/RT0805BR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
- R30: renamed from R32; Manufactor Part Number (none) -> RC0603JR-070RL; Supplier Part Number (none) -> 311-0.0GRCT-ND; Supplier link (none) -> https://www.digikey.co.nz/en/products/detail/yageo/RC0603JR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
- R31: renamed from R33; Manufactor Part Number (none) -> RC0603JR-070RL; Supplier Part Number (none) -> 311-0.0GRCT-ND; Supplier link (none) -> https://www.digikey.co.nz/en/products/detail/yageo/RC0603JR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
- R32: renamed from R34; Manufactor Part Number (none) -> RC0603JR-070RL; Supplier Part Number (none) -> 311-0.0GRCT-ND; Supplier link (none) -> https://www.digikey.co.nz/en/products/detail/yageo/RC0603JR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
- R33: renamed from R35; Manufactor Part Number (none) -> RC0603JR-070RL; Supplier Part Number (none) -> 311-0.0GRCT-ND; Supplier link (none) -> https://www.digikey.co.nz/en/products/detail/yageo/RC0603JR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
- R4: Manufactor Part Number (none) -> RT0603BRD07158RL; Notes (none) -> 25ppm; Supplier Part Number (none) -> YAG4477CT-ND; Supplier link (none) -> https://www.digikey.co.nz/en/products/detail/yageo/RT0603BR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
- R5: Manufactor Part Number (none) -> RT0603DRD0715RL; Notes (none) -> 25ppm; Supplier Part Number (none) -> 13-RT0603DRD0715RLCT-ND; Supplier link (none) -> https://www.digikey.co.nz/en/products/detail/yageo/RT0603DR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
- R7: renamed from R9; Manufactor Part Number (none) -> RT0603BRD0710KL; Supplier Part Number (none) -> YAG1236CT-ND; Supplier link (none) -> https://www.digikey.co.nz/en/products/detail/yageo/RT0603BR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
- R8: renamed from R10; Manufactor Part Number (none) -> RT0603BRD0710KL; Supplier Part Number (none) -> YAG1236CT-ND; Supplier link (none) -> https://www.digikey.co.nz/en/products/detail/yageo/RT0603BR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
- R9: renamed from R11; Manufactor Part Number (none) -> RT0603BRD0710KL; Supplier Part Number (none) -> YAG1236CT-ND; Supplier link (none) -> https://www.digikey.co.nz/en/products/detail/yageo/RT0603BR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
- renumbered C6 to C10, C7 to C11, C8 to C12, C9 to C13, C10 to C14, C11 to C15, C12 to C16, C13 to C17, C14 to C18, C15 to C19, C16 to C20, C17 to C21, C18 to C22, C19 to C23, C20 to C24, C21 to C25, C22 to C26, C23 to C27, C1 to C3, C2 to C4, C3 to C5, C4 to C8, C5 to C9, R6 to R12, R8 to R6, RxL to RxL1, RxO to RxO1, RxS to RxS1
Connections:
- net VCC: now also FB5.1; no longer C1.1, C2.1, C3.1, C4.1, C5.1, J5.3 (Pin_3), U1.7 (V+)
- net VS: now also FB4.1; no longer C10.1, C6.1, C7.1, C8.1, C9.1, U1.4 (V-)
- new net: C10.1, C6.1, C7.1, C8.1, C9.1, FB4.2, U1.4 (V-)
- new net: C1.1, C2.1, C3.1, C4.1, C5.1, FB5.2, J5.3 (Pin_3), U1.7 (V+)
Other:
- note added: "AMP INTERNALS"
- note added: "BNC"
- note added: "FUNCTION GEN"
- note added: "FUNCTIONAL DIAGRAM OF SYSTEM INPUT"
- note removed: "FUNCTIONAL DIAGRAM OF SYSTEM"
- moved on the sheet: C10, C6, C7, C8, C9

Commit message: updated title block
Other:
- company: (none) -> sirlilpanda
- title: (none) -> SCOPE CREEP AMP
Changed lines of the file:
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@@
 	(generator_version "9.0")
 	(paper "A3")
+	(title_block
+		(title "SCOPE CREEP AMP")
+		(date "2025-08-21")
+		(rev "REV: A")
+		(company "sirlilpanda")
+		(comment 1 "DESGINER: LOGAN HENDERSON")
+	)
 	(rectangle
 		(start 63.5 60.96)
